Commit message: Part 1: add meshes and modify launch files

File: urdf/tb3_burger.urdf (robot description, URDF)
Before this commit: robot tb3_burger, 34 links, 33 joints
Links:
- link lidar_spinner_link: geometry collision cylinder length=0.0188 radius=0.0327; visual mesh filename=package://ros2_urdf_project/meshes/lds_top.dae scale=0.001 0.001 0.001
- link lidar_support_link: geometry collision box size=0.0947 0.0727 0.0257; visual mesh filename=package://ros2_urdf_project/meshes/lds_base.dae scale=0.001 0.001 0.001
Joints:
- joint left_wheel_joint: origin xyz=-0.015 -0.026 0 rpy=1.571 0 0 -> xyz=-0.015 -0.0259 0 rpy=1.571 0 0
- joint lidar_spinner_joint: origin xyz=0 0 0.02225 rpy=0 0 0 -> xyz=0 0 0.02225 rpy=0 0 3.142
- joint lidar_support_joint: origin xyz=0 0 0.01735 rpy=0 0 0 -> xyz=0 0 0.01735 rpy=0 0 3.142
- joint right_wheel_joint: origin xyz=-0.015 0.026 0 rpy=1.571 0 0 -> xyz=-0.015 0.0259 0 rpy=1.571 0 0

Commit message: Part 1: update caster wheel

File: urdf/tb3_burger.urdf (robot description, URDF)
Before this commit: robot tb3_burger, 34 links, 33 joints
Links:
- removed link caster_wheel_link
- link caster_pitch_link: mass None -> 0.010; geometry collision sphere radius=0.005; visual sphere radius=0.005
- link caster_roll_link: mass None -> 0.001; geometry collision cylinder length=0.001 radius=0.0045000000000000005; visual cylinder length=0.001 radius=0.0045000000000000005
- link caster_yaw_link: mass None -> 0.001; geometry collision cylinder length=0.001 radius=0.0045000000000000005; visual cylinder length=0.001 radius=0.0045000000000000005
- link lidar_spinner_link: geometry collision cylinder length=0.0188 radius=0.0327; visual cylinder length=0.0188 radius=0.0327
- link lidar_support_link: geometry collision box size=0.0947 0.0727 0.0257; visual box size=0.0947 0.0727 0.0257
Joints:
- removed joint caster_wheel_joint
- joint left_wheel_joint: axis 1 0 0 -> 0 1 0; origin xyz=-0.015 -0.0259 0 rpy=1.571 0 0 -> xyz=-0.012 -0.0259 0 rpy=0 1.571 1.571
- joint lidar_spinner_joint: axis (none) -> 0 0 1; limit (none) -> effort=10.0 velocity=2.0; origin xyz=0 0 0.02225 rpy=0 0 3.142 -> xyz=0 0 0.02225 rpy=0 0 0; type fixed -> continuous
- joint right_wheel_joint: axis 1 0 0 -> 0 1 0; origin xyz=-0.015 0.0259 0 rpy=1.571 0 0 -> xyz=-0.012 0.0259 0 rpy=0 1.571 1.571

Commit message: Part 1: add camera

File: urdf/tb3_burger.urdf (robot description, URDF)
Before this commit: robot tb3_burger, 33 links, 32 joints
Links:
- added link camera_link, mass 0.010; collision box size=0.005 0.030 0.030; visual box size=0.005 0.030 0.030
- added link camera_support_link, mass 0.010; collision box size=0.005 0.030 0.015; visual box size=0.005 0.030 0.015
Joints:
- added joint camera_joint: type fixed, parent camera_support_link, child camera_link, origin xyz=-0.005 0 -0.0075 rpy=0 0 0
- added joint camera_support_joint: type fixed, parent chassis_plate_3_link, child camera_support_link, origin xyz=-0.06625 0 0.01 rpy=0 0 0
- joint spacer35_3_joint: origin xyz=-0.06375 -0.015 0.018 rpy=0 0 0 -> xyz=-0.06375 -0.0125 0.018 rpy=0 0 0
- joint spacer35_4_joint: origin xyz=-0.06375 0.015 0.018 rpy=0 0 0 -> xyz=-0.06375 0.0125 0.018 rpy=0 0 0

Commit message: Part 1: add gazebo colors

File: urdf/tb3_burger.urdf (robot description, URDF)
Before this commit: robot tb3_burger, 35 links, 34 joints
Links:
- removed link caster_pitch_link
- removed link caster_roll_link
- removed link caster_yaw_link
- added link caster_wheel_pitch_link, mass 0.010; collision sphere radius=0.005; visual sphere radius=0.005
- added link caster_wheel_roll_link, mass 0.001; collision cylinder length=0.001 radius=0.0045000000000000005; visual cylinder length=0.001 radius=0.0045000000000000005
- added link caster_wheel_yaw_link, mass 0.001; collision cylinder length=0.001 radius=0.0045000000000000005; visual cylinder length=0.001 radius=0.0045000000000000005
Joints:
- removed joint caster_pitch_joint
- removed joint caster_roll_joint
- removed joint caster_yaw_joint
- added joint caster_wheel_pitch_joint: type continuous, parent caster_wheel_roll_link, child caster_wheel_pitch_link, origin xyz=0 0 0 rpy=0 0 0, axis 0 1 0, limit effort=1000.0 velocity=100.0
- added joint caster_wheel_roll_joint: type continuous, parent caster_wheel_yaw_link, child caster_wheel_roll_link, origin xyz=0 0 0 rpy=0 0 0, axis 1 0 0, limit effort=1000.0 velocity=100.0
- added joint caster_wheel_yaw_joint: type continuous, parent caster_wheel_support_link, child caster_wheel_yaw_link, origin xyz=0 0 -0.004 rpy=0 0 0, axis 0 0 1, limit effort=1000.0 velocity=100.0

Commit message: Part2: add joint state publisher and differential drive, fix urdf elements position

File: urdf/tb3_burger.urdf (robot description, URDF)
Before this commit: robot tb3_burger, 35 links, 34 joints
Links:
- removed link lidar_usb_board_link
- added link imu_chip_link, mass 0.002; collision box size=0.005 0.005 0.0025; visual box size=0.005 0.005 0.0025
Joints:
- removed joint lidar_usb_board_joint
- added joint imu_chip_joint: type fixed, parent chassis_plate_3_link, child imu_chip_link, origin xyz=0.015 0 0.00675 rpy=0 0 0
- joint battery_joint: origin xyz=-0.011625 0 0.01825 rpy=0 0 0 -> xyz=0.011625 0 0.01825 rpy=0 0 0
- joint camera_joint: origin xyz=-0.005 0 -0.0075 rpy=0 0 0 -> xyz=0.005 0 -0.0075 rpy=0 0 0
- joint camera_support_joint: origin xyz=-0.06625 0 0.01 rpy=0 0 0 -> xyz=0.06625 0 0.01 rpy=0 0 0
- joint caster_wheel_support_joint: origin xyz=0.04875 0 -0.0085 rpy=0 0 0 -> xyz=-0.04875 0 -0.0085 rpy=0 0 0
- joint drive_motor_1_joint: origin xyz=-0.0255 0.05175 0.01875 rpy=0 0 0 -> xyz=0.0255 0.05175 0.01875 rpy=0 0 0
- joint drive_motor_2_joint: origin xyz=-0.0255 -0.05175 0.01875 rpy=0 0 0 -> xyz=0.0255 -0.05175 0.01875 rpy=0 0 0
- joint left_wheel_joint: axis 0 1 0 -> 0 0 1; origin xyz=-0.012 -0.0259 0 rpy=0 1.571 1.571 -> xyz=0.012 -0.0259 0 rpy=0 1.571 1.571
- joint raspi_board_joint: origin xyz=0.030 0 0.01475 rpy=0 0 0 -> xyz=-0.030 0 0.01475 rpy=0 0 0
- joint right_wheel_joint: axis 0 1 0 -> 0 0 1; origin xyz=-0.012 0.0259 0 rpy=0 1.571 1.571 -> xyz=0.012 0.0259 0 rpy=0 1.571 1.571
- joint spacer35_1_joint: origin xyz=0.024 -0.06375 0.018 rpy=0 0 0 -> xyz=-0.024 -0.06375 0.018 rpy=0 0 0
- joint spacer35_2_joint: origin xyz=0.024 0.06375 0.018 rpy=0 0 0 -> xyz=-0.024 0.06375 0.018 rpy=0 0 0
- joint spacer35_3_joint: origin xyz=-0.06375 -0.0125 0.018 rpy=0 0 0 -> xyz=0.06375 -0.0125 0.018 rpy=0 0 0
- joint spacer35_4_joint: origin xyz=-0.06375 0.0125 0.018 rpy=0 0 0 -> xyz=0.06375 0.0125 0.018 rpy=0 0 0
- joint spacer45_10_joint: origin xyz=-0.024 0.06375 0.018 rpy=0 0 0 -> xyz=0.024 0.06375 0.018 rpy=0 0 0
- joint spacer45_1_joint: origin xyz=0.06375 -0.025 0.018 rpy=0 0 0 -> xyz=-0.06375 -0.025 0.018 rpy=0 0 0
- joint spacer45_2_joint: origin xyz=0.06375 0.025 0.018 rpy=0 0 0 -> xyz=-0.06375 0.025 0.018 rpy=0 0 0
- joint spacer45_3_joint: origin xyz=-0.06375 -0.025 0.018 rpy=0 0 0 -> xyz=0.06375 -0.025 0.018 rpy=0 0 0
- joint spacer45_4_joint: origin xyz=-0.06375 0.025 0.018 rpy=0 0 0 -> xyz=0.06375 0.025 0.018 rpy=0 0 0
- joint spacer45_7_joint: origin xyz=-0.06375 -0.025 0.018 rpy=0 0 0 -> xyz=0.06375 -0.025 0.018 rpy=0 0 0
- joint spacer45_8_joint: origin xyz=-0.06375 0.025 0.018 rpy=0 0 0 -> xyz=0.06375 0.025 0.018 rpy=0 0 0
- joint spacer45_9_joint: origin xyz=-0.024 -0.06375 0.018 rpy=0 0 0 -> xyz=0.024 -0.06375 0.018 rpy=0 0 0

Commit message: Part 2: fix left and right wheels position

File: urdf/tb3_burger.urdf (robot description, URDF)
Before this commit: robot tb3_burger, 35 links, 34 joints
Joints:
- joint left_wheel_joint: origin xyz=0.012 -0.0259 0 rpy=0 1.571 1.571 -> xyz=0.012 0.0259 0 rpy=0 1.571 1.571; parent drive_motor_2_link -> drive_motor_1_link
- joint right_wheel_joint: origin xyz=0.012 0.0259 0 rpy=0 1.571 1.571 -> xyz=0.012 -0.0259 0 rpy=0 1.571 1.571; parent drive_motor_1_link -> drive_motor_2_link
